File: hw/AES-DAC/AES-DAC.kicad_pcb (KiCad board)
At the start: 2 copper layers, 96 x 74 mm, 129 parts, among them J1 XLR3, J2 XLR3, J3 XLR3, J4 DCJ200-10-A-K1-K, T1 PE-65812NLT, U1 DIR9001, U2 OPA1612AxD, U3 PCM1789, U4 APX803S05-29SA-7, U5 OPA1612AxD, U6 TPS7A49, U7 TPS7A49

Commit message: layout update
Parts:
- added C39: 100u, Capacitor_SMD:CP_Elec_6.3x7.7, F.Cu at (64.5, 74.0)
- added C46: 100u, Capacitor_SMD:CP_Elec_6.3x7.7, F.Cu at (64.5, 86.5)
- added J4: TestPoint_Small, TestPoint:TestPoint_THTPad_D2.0mm_Drill1.0mm, F.Cu at (114.0, 90.5)
- added J5: TestPoint_Small, TestPoint:TestPoint_THTPad_D2.0mm_Drill1.0mm, F.Cu at (114.0, 23.0)
- C15, C17, C18, C19, C20, C21, C22, C23, C24, FB1, FB2, FB3, FB4, R29, R31: moved to B.Cu
- R32, R37: footprint Resistor_SMD:R_0805_2012Metric_Pad1.20x1.40mm_HandSolder -> Resistor_SMD:R_0603_1608Metric_Pad0.98x0.95mm_HandSolder
- TP1, TP2, TP4, TP5, TP7, TP8, TP9: footprint TestPoint:TestPoint_Pad_D1.5mm -> TestPoint:TestPoint_Pad_D1.0mm; moved to B.Cu
- TP3, TP6: footprint TestPoint:TestPoint_Pad_D1.5mm -> TestPoint:TestPoint_Pad_D1.0mm
- moved U4 146.2 mm to (44.0, 52.1), turned to -90 degrees
- moved R9 142.7 mm to (43.0, 65.5), turned to 90 degrees
- moved TP8 142.6 mm to (45.2, 47.5), turned to 90 degrees
- moved TP7 142.6 mm to (45.2, 44.0), turned to 90 degrees
- moved R3 142.4 mm to (43.0, 61.5), turned to -90 degrees
- moved R5 141.4 mm to (40.5, 65.5)
- moved R1 140.3 mm to (40.5, 57.4)
- moved TP4 139.3 mm to (45.5, 40.0), turned to 180 degrees
- moved TP1 137.5 mm to (43.0, 46.0), turned to 90 degrees
- moved R4 137.1 mm to (40.5, 61.5)
- moved TP6 136.1 mm to (54.5, 22.5), turned to -90 degrees
- moved TP3 134.9 mm to (52.2, 22.5), turned to -90 degrees
- moved TP9 132.2 mm to (57.0, 42.0), turned to 180 degrees
- moved C21 131.7 mm to (49.8, 48.5)
- moved C23 131.4 mm to (49.8, 37.5)
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- renumbered C39 to C40, C40 to C41, C41 to C42, C42 to C43, C43 to C44, C44 to C45, C45 to C47, J4 to J6
Connections:
- net Net-(C32-Pad1) renamed /VIN
- net Net-(U3A-VOUTL+) renamed /VOUTL+
- net Net-(U3A-VOUTL-) renamed /VOUTL-
- C12 pad 1: /XLR_R_- -> /XLR_R_+
- C28 pad 1: /XLR_R_+ -> /XLR_R_-
- J3 pad 2: /XLR_R_- -> /XLR_R_+
- J3 pad 3: /XLR_R_+ -> /XLR_R_-
- R41 pad 1: Net-(U3A-VOUTR+) -> /VOUTR-
- R46 pad 1: Net-(U3A-VOUTR-) -> /VOUTR+
- U3 pad 13: Net-(U3A-VOUTR+) -> /VOUTR+
- U3 pad 14: Net-(U3A-VOUTR-) -> /VOUTR-
Routing:
- net /VOUTL+: track 0.00 -> 57.1 mm
- net /AMUTE: track 0.00 -> 39.4 mm, vias 0 -> 2
- net /VOUTR+: track 0.00 -> 39.3 mm
- net /VOUTL-: track 0.00 -> 37.7 mm
- net /Vcom: track 0.00 -> 35.6 mm, vias 0 -> 4
- net /RSTN: track 0.00 -> 29.4 mm
- net +5V: track 0.00 -> 23.2 mm, vias 0 -> 2
- net /DEMP: track 0.00 -> 22.7 mm, vias 0 -> 2
- net Net-(U1C-PSCK0): track 0.00 -> 21.0 mm, vias 0 -> 2
- net Net-(U1B-RXIN): track 0.00 -> 20.3 mm, vias 0 -> 1
- net Net-(U1C-PSCK1): track 0.00 -> 20.2 mm, vias 0 -> 2
- net Net-(C2-Pad1): track 0.00 -> 19.3 mm
- net Net-(C11-Pad1): track 0.00 -> 19.3 mm
- net +3.3V: track 0.00 -> 19.0 mm
- net Net-(C7-Pad1): track 0.00 -> 17.9 mm
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- added copper zone on B.Cu, net +5V
- added copper zone on F.Cu, net /VIN
- added copper zone on F.Cu, net Earth
Other:
- copper layers 2 -> 4

Commit message: layout update
Parts:
- removed the FB2 at (59.5, 33.5)
- added D1: LED, LED_THT:LED_D3.0mm_Horizontal_O3.81mm_Z6.0mm, F.Cu at (24.2, 70.7)
- added G***: LOGO, others:Logo_20mm, F.Cu at (78.4, 85.7)
- added Q1: BC857, Package_TO_SOT_SMD:SOT-23, F.Cu at (45.8, 67.0)
- added R51: 0R, Resistor_SMD:R_0805_2012Metric_Pad1.20x1.40mm_HandSolder, F.Cu at (97.5, 24.8)
- added R52: 0R, Resistor_SMD:R_0805_2012Metric_Pad1.20x1.40mm_HandSolder, F.Cu at (97.5, 88.8)
- added R55: 1k, Resistor_SMD:R_0603_1608Metric_Pad0.98x0.95mm_HandSolder, F.Cu at (46.7, 62.2)
- added R57: 220R, Resistor_SMD:R_0805_2012Metric_Pad1.20x1.40mm_HandSolder, F.Cu at (28.0, 70.0)
- added SW1: SW_DIP_x01, Button_Switch_SMD:SW_DIP_SPSTx01_Slide_6.7x4.1mm_W6.73mm_P2.54mm_LowProfile_JPin, B.Cu at (35.2, 45.8)
- TP1, TP2, TP5, TP7, TP8, TP9: moved to F.Cu
- moved FB1 8.63 mm to (47.5, 42.0), turned to 90 degrees
- moved TP1 8.27 mm to (43.5, 54.2)
- moved TP7 7.28 mm to (41.5, 50.2)
- moved TP4 6.35 mm to (48.5, 45.6)
- moved R37 5.83 mm to (57.3, 64.5)
- moved R20 5.83 mm to (57.3, 60.5)
- moved R35 5.74 mm to (49.8, 64.5)
- moved R36 5.74 mm to (52.3, 64.5)
- moved R38 5.74 mm to (54.8, 64.5)
- moved R39 5.74 mm to (59.8, 64.5)
- moved C17 5.74 mm to (56.9, 30.5)
- moved C19 5.74 mm to (56.9, 28.0)
- moved R13 5.74 mm to (48.1, 41.0)
- moved C15 5.74 mm to (52.3, 39.0)
- moved C16 5.74 mm to (52.3, 36.5)
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- renumbered C24 to C23, C23 to C24, FB3 to FB2, FB4 to FB3, R52 to R53, R53 to R54, R51 to R56, R54 to R58, R55 to R59, R56 to R60, R57 to R61
Connections:
- C17 pad 2: Net-(U3B-VCC1) -> +5V
- C18 pad 2: Net-(U3B-VCC1) -> +5V
- C19 pad 2: Net-(U3B-VCC1) -> +5V
- C20 pad 2: Net-(U3B-VCC1) -> +5V
- J1 pad 1: Net-(J1-Pad1) -> /EARTH_AES
- U3 pad 16: Net-(U3B-VCC1) -> +5V
- U3 pad 8: Net-(U3B-VCC1) -> +5V
Routing:
- net GND: track 0.00 -> 93.3 mm, vias 0 -> 285
- net Net-(J1-Pad3): track 0.00 -> 38.7 mm, vias 0 -> 1
- net Net-(D1-A): track 0.00 -> 29.7 mm
- net +3.3V: track 19.0 -> 41.8 mm, vias 0 -> 21
- net Net-(C1-Pad1): track 0.00 -> 22.4 mm, vias 0 -> 1
- net +5V: track 23.2 -> 42.9 mm, vias 2 -> 27
- net Net-(U3B-VCC1): track 11.0 -> 0.00 mm, vias 2 -> 0
- net /VOUTR+: track 39.3 -> 28.5 mm
- net Net-(U1B-BFRAME): track 0.00 -> 10.8 mm, vias 0 -> 2
- net Net-(R4-Pad2): track 0.00 -> 10.0 mm
- net Net-(R1-Pad1): track 0.00 -> 8.80 mm
- net Net-(U1C-FSOUT1): track 0.00 -> 7.81 mm
- net /VOUTL-: track 37.7 -> 30.3 mm
- net Net-(U7-EN): track 2.50 -> 9.78 mm, vias 0 -> 2
- net /VOUTL+: track 57.1 -> 49.8 mm
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- added copper zone on B.Cu, net +3.3V
- added copper zone on F.Cu, net +3.3V
- added copper zone on F.Cu, net +5V
- added copper zone on B.Cu, net /EARTH_AES
- added copper zone on F.Cu, net /EARTH_AES
- added copper zone on In1.Cu, net /EARTH_AES
- added copper zone on In2.Cu, net /EARTH_AES
- added copper zone on In2.Cu, net /Vcom
- added copper zone on B.Cu, net Earth
- added copper zone on In1.Cu, net Earth
- added copper zone on In2.Cu, net Earth
- added copper zone on B.Cu, net GND
- added copper zone on F.Cu, net GND
- added copper zone on In1.Cu, net GND
- added copper zone on In2.Cu, net GND
- added copper zone on B.Cu, net Net-(U3B-VDD)
Other:
- board text added: "AES - DAC 2024 - Rev A"
- board text added: "GND Lift"
- board text added: "Left"
- board text added: "Right"

Commit message: Added Gerbers and did some improvements
Parts:
- added D1: PESD5V0U1UB, Diode_SMD:D_SOD-523, B.Cu at (91.5, 60.5)
- added D2: PESD5V0U1UB, Diode_SMD:D_SOD-523, B.Cu at (91.5, 84.0)
- added D3: PESD5V0U1UB, Diode_SMD:D_SOD-523, B.Cu at (91.5, 29.8)
- added D4: PESD5V0U1UB, Diode_SMD:D_SOD-523, B.Cu at (91.5, 53.5)
- added D6: PMEG4010CEH, Diode_SMD:D_SOD-123F, F.Cu at (35.2, 88.2)
- C6: footprint Capacitor_SMD:C_1206_3216Metric_Pad1.33x1.80mm_HandSolder -> Capacitor_SMD:C_0805_2012Metric_Pad1.18x1.45mm_HandSolder
- Q1: value BC857 -> BC847
- moved C6 0.28 mm to (56.0, 33.0)
- renumbered C33 to C32, C34 to C33, C32 to C34, D1 to D5, R51 to R49, R49 to R50, R50 to R51, R56 to R53, R53 to R54, R54 to R55, R57 to R56, R55 to R57
Connections:
- D5 pad 2: Net-(D1-A) -> +3.3V
- J6 pad 2: /VIN -> Net-(D6-A)
- J6 pad 3: /VIN -> Net-(D6-A)
- Q1 pad 2: +3.3V -> GND
- Q1 pad 3: Net-(D1-A) -> Net-(Q1-C)
- R56 pad 1: GND -> Net-(Q1-C)
Routing:
- net Net-(D1-A): track 29.7 -> 0.00 mm
- net +3.3V: track 41.8 -> 66.9 mm
- net Net-(Q1-C): track 0.00 -> 18.1 mm
- net Net-(D6-A): track 0.00 -> 15.2 mm
- net GND: track 93.3 -> 98.3 mm, vias 285 -> 289
- net Net-(C8-Pad2): track 7.00 -> 9.30 mm
- net Net-(C28-Pad2): track 7.00 -> 9.30 mm
- net Net-(C12-Pad2): track 7.00 -> 9.24 mm
- net Net-(C3-Pad2): track 7.00 -> 9.19 mm
- net /Vcom: track 40.7 -> 41.3 mm
Other:
- board text added: "AES - DAC 2025 - Rev A"
- board text removed: "AES - DAC 2024 - Rev A"
