File: hw/AES-DAC/AES-DAC.kicad_sch (KiCad schematic)
At the start: 126 parts

Commit message: minor corrections in schematic
Parts:
- removed C? (x4): 1u, symbol Device:C_Small
- removed C?: 10n, symbol Device:C_Small
- removed C? (x7): 10u, symbol Device:C_Polarized_Small
- removed FB? (x2): FerriteBead_Small, symbol Device:FerriteBead_Small
- added C? (x7): 10u, symbol Device:C_Small
- added C?: 10n, symbol Device:C_Small
- added C?: 100u, symbol Device:C_Polarized_Small
- added C?: 1u, symbol Device:C_Small
- added C? (x3): 100n, symbol Device:C_Small
- added FB? (x2): FerriteBead_Small, symbol Device:FerriteBead_Small
- added R? (x2): 0R, Resistor_SMD:R_0805_2012Metric_Pad1.20x1.40mm_HandSolder, symbol Device:R_Small
- added R?: 4.7k, Resistor_SMD:R_0805_2012Metric_Pad1.20x1.40mm_HandSolder, symbol Device:R_Small
- added TP? (x2): TestPoint_Small, TestPoint:TestPoint_Pad_D1.5mm, symbol Connector:TestPoint_Small
- C?: value C_Small -> 100n
- C? (x4): value 220p -> 22u
- C?: value 1u -> 100n
- R? (x12): value 0R -> 4.7k
- R? (x2): now not fitted
- T?: value Transformer_1P_1S -> PE-65812NLT
- U? (x2): LCSC Part (none) -> C16430
- U? (x5): LCSC Part (none) -> C94590
Connections:
- net +3.3V: now also C?.2, C?.2, FB?.1, FB?.1, R?.1
- net +5V: now also C?.2, C?.2
- net Earth: now also SW?.1, R?.2
- net GND: now also C?.1, C?.1, C?.1, C?.1, C?.1, C?.1, C?.1, C?.1, C?.1, C?.1, C?.1, C?.1, C?.2, R?.1; no longer SW?.1
- net RSTN: now also R?.1; no longer U?.4 (~{RST})
- net at C?.2, FB?.2, U?.6 (VDD): now also C?.2
- net at C?.2, C?.2, U?.5 (VDD): now also FB?.2
- net at U?.6 (NR/SS): now also C?.2
- net at C?.2, L?.2, R?.1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: now also C?.2
- net at C?.2, FB?.2, U?.16 (VCC2)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: now also C?.2, C?.2, C?.2
- net at C?.2, C?.2, U?.24 (VCC): now also FB?.2
- net at L?.2, R?.1, U?.8 (IN): now also C?.2, C?.2
- net at J?.2, J?.3, L?.1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: now also C?.1
- net at U?.18 (ZERO2): now also TP?.1
- net at U?.19 (ZERO1): now also TP?.1
- new net: R?.2, R?.2, U?.4 (~{RST})
Other:
- note added: "Circuit for FILT as recommended in Datasheet"
- note added: "PCM1789 does not require particular power sequence"
- note added: "RSV: Pull to GND in HW-Mode FMT: Pull to GND for I2S format SCKI: supported 128 fS, 192 fS, 256 fS, 384 fS, 512 fS, 768 fS, and 1152 fS FMT: 220k Pull-Down for HW-Mode"
- note added: "Vout = 4 Vpp,"
- note added: "Vout = 8 Vpp (diff)"
- note removed: "PCM1789 does not require particular power-on sequences"
- note removed: "RSV: Pull to GND in HW-Mode FMT: Pull to GND for I2S format SCKI: supported 128 fS, 192 fS, 256 fS, 384 fS, 512 fS, 768 fS, and 1152 fS"
- moved on the sheet: C?, FB?, J?, L?, R?, U?, U?A, U?B

Commit message: Annotated schematic
Parts:
- gave numbers to parts that had none: 125

Commit message: Added: Simulation for Jitter analysis PCB File Updated: Schematic
Parts:
- removed T1: PE-65812NLT, symbol Device:Transformer_1P_1S
- added R1, R3, R5, R9: 0R, Resistor_SMD:R_0603_1608Metric_Pad0.98x0.95mm_HandSolder, symbol Device:R_Small
- added T1: PE-65812NLT, components:PE-65812NLT, symbol SimonLib:PE-65812NLT
- added TP1: TestPoint_Small, TestPoint:TestPoint_Pad_D1.5mm, symbol Connector:TestPoint_Small
- C1, C10, C14, C15, C16, C17, C18, C19, C20, C21, C22, C23, C24, C30, C33, C34, C35, C36, C37, C38, C41, C42, C43, C44, C5: footprint (none) -> Capacitor_SMD:C_0805_2012Metric_Pad1.18x1.45mm_HandSolder
- C11, C13, C2, C26, C29, C4, C7, C9: footprint (none) -> Capacitor_THT:C_Rect_L7.2mm_W4.5mm_P5.00mm_FKS2_FKP2_MKS2_MKP2
- C12, C28: footprint (none) -> Capacitor_THT:C_Radial_D10.0mm_H12.5mm_P5.00mm
- C25: footprint (none) -> Capacitor_SMD:C_0805_2012Metric_Pad1.18x1.45mm_HandSolder; LCSC Part (none) -> C77063
- C27: footprint (none) -> Capacitor_SMD:C_0805_2012Metric_Pad1.18x1.45mm_HandSolder; LCSC Part (none) -> C77084
- C3, C8: footprint (none) -> Capacitor_THT:C_Radial_D10.0mm_H12.5mm_P5.00mm; TME Part (none) -> UES1E470MPM
- C31, C40: footprint (none) -> Capacitor_SMD:C_0805_2012Metric_Pad1.18x1.45mm_HandSolder; LCSC Part (none) -> C97905
- C32: footprint (none) -> Capacitor_SMD:CP_Elec_6.3x7.7; LCSC Part (none) -> C134220
- C39, C45: footprint (none) -> Capacitor_SMD:C_0805_2012Metric_Pad1.18x1.45mm_HandSolder; Dielektrikum (none) -> C0G; LCSC Part (none) -> C97905
- C6: footprint (none) -> Capacitor_SMD:C_1206_3216Metric_Pad1.33x1.80mm_HandSolder
- FB1, FB2, FB3, FB4: footprint (none) -> Resistor_SMD:R_0805_2012Metric_Pad1.20x1.40mm_HandSolder
- J1: footprint (none) -> Connector_Audio:Jack_XLR_Neutrik_NC3FAH1-0_Horizontal
- J2, J3: footprint (none) -> Connector_Audio:Jack_XLR_Neutrik_NC3MAH-0_Horizontal
- L1, L2: footprint (none) -> Inductor_SMD:L_1206_3216Metric
- R10: renamed from R6; footprint Resistor_SMD:R_0805_2012Metric_Pad1.20x1.40mm_HandSolder -> Resistor_SMD:R_0603_1608Metric_Pad0.98x0.95mm_HandSolder
- R12: renamed from R8; footprint Resistor_SMD:R_0805_2012Metric_Pad1.20x1.40mm_HandSolder -> Resistor_SMD:R_0603_1608Metric_Pad0.98x0.95mm_HandSolder
- R13: renamed from R9; footprint Resistor_SMD:R_0805_2012Metric_Pad1.20x1.40mm_HandSolder -> Resistor_SMD:R_0603_1608Metric_Pad0.98x0.95mm_HandSolder
- R14: renamed from R10; footprint Resistor_SMD:R_0805_2012Metric_Pad1.20x1.40mm_HandSolder -> Resistor_SMD:R_0603_1608Metric_Pad0.98x0.95mm_HandSolder
- R15: renamed from R11; footprint Resistor_SMD:R_0805_2012Metric_Pad1.20x1.40mm_HandSolder -> Resistor_SMD:R_0603_1608Metric_Pad0.98x0.95mm_HandSolder
- R17: renamed from R13; footprint Resistor_SMD:R_0805_2012Metric_Pad1.20x1.40mm_HandSolder -> Resistor_SMD:R_0603_1608Metric_Pad0.98x0.95mm_HandSolder
- R18: renamed from R14; footprint Resistor_SMD:R_0805_2012Metric_Pad1.20x1.40mm_HandSolder -> Resistor_SMD:R_0603_1608Metric_Pad0.98x0.95mm_HandSolder
- R19: renamed from R15; footprint Resistor_SMD:R_0805_2012Metric_Pad1.20x1.40mm_HandSolder -> Resistor_SMD:R_0603_1608Metric_Pad0.98x0.95mm_HandSolder
- R20: renamed from R16; footprint Resistor_SMD:R_0805_2012Metric_Pad1.20x1.40mm_HandSolder -> Resistor_SMD:R_0603_1608Metric_Pad0.98x0.95mm_HandSolder
- R21: renamed from R17; footprint Resistor_SMD:R_0805_2012Metric_Pad1.20x1.40mm_HandSolder -> Resistor_SMD:R_0603_1608Metric_Pad0.98x0.95mm_HandSolder
- R22: renamed from R18; footprint Resistor_SMD:R_0805_2012Metric_Pad1.20x1.40mm_HandSolder -> Resistor_SMD:R_0603_1608Metric_Pad0.98x0.95mm_HandSolder
- R25: renamed from R21; footprint Resistor_SMD:R_0805_2012Metric_Pad1.20x1.40mm_HandSolder -> Resistor_SMD:R_0603_1608Metric_Pad0.98x0.95mm_HandSolder
- R26: renamed from R22; footprint Resistor_SMD:R_0805_2012Metric_Pad1.20x1.40mm_HandSolder -> Resistor_SMD:R_0603_1608Metric_Pad0.98x0.95mm_HandSolder
- R27: renamed from R23; footprint Resistor_SMD:R_0805_2012Metric_Pad1.20x1.40mm_HandSolder -> Resistor_SMD:R_0603_1608Metric_Pad0.98x0.95mm_HandSolder
- R28: renamed from R24; footprint Resistor_SMD:R_0805_2012Metric_Pad1.20x1.40mm_HandSolder -> Resistor_SMD:R_0603_1608Metric_Pad0.98x0.95mm_HandSolder
- R29: renamed from R25; footprint Resistor_SMD:R_0805_2012Metric_Pad1.20x1.40mm_HandSolder -> Resistor_SMD:R_0603_1608Metric_Pad0.98x0.95mm_HandSolder
- R31: renamed from R27; footprint Resistor_SMD:R_0805_2012Metric_Pad1.20x1.40mm_HandSolder -> Resistor_SMD:R_0603_1608Metric_Pad0.98x0.95mm_HandSolder
- R33: renamed from R29; footprint Resistor_SMD:R_0805_2012Metric_Pad1.20x1.40mm_HandSolder -> Resistor_SMD:R_0603_1608Metric_Pad0.98x0.95mm_HandSolder
- R34: renamed from R30; footprint Resistor_SMD:R_0805_2012Metric_Pad1.20x1.40mm_HandSolder -> Resistor_SMD:R_0603_1608Metric_Pad0.98x0.95mm_HandSolder
- R35: renamed from R31; footprint Resistor_SMD:R_0805_2012Metric_Pad1.20x1.40mm_HandSolder -> Resistor_SMD:R_0603_1608Metric_Pad0.98x0.95mm_HandSolder
- R36: renamed from R32; footprint Resistor_SMD:R_0805_2012Metric_Pad1.20x1.40mm_HandSolder -> Resistor_SMD:R_0603_1608Metric_Pad0.98x0.95mm_HandSolder
- R38: renamed from R34; footprint Resistor_SMD:R_0805_2012Metric_Pad1.20x1.40mm_HandSolder -> Resistor_SMD:R_0603_1608Metric_Pad0.98x0.95mm_HandSolder
- R39: renamed from R35; footprint Resistor_SMD:R_0805_2012Metric_Pad1.20x1.40mm_HandSolder -> Resistor_SMD:R_0603_1608Metric_Pad0.98x0.95mm_HandSolder
- R4: renamed from R2; footprint (none) -> Capacitor_SMD:C_0805_2012Metric_Pad1.18x1.45mm_HandSolder
- R6: renamed from R3; footprint Resistor_SMD:R_0805_2012Metric_Pad1.20x1.40mm_HandSolder -> Resistor_SMD:R_0603_1608Metric_Pad0.98x0.95mm_HandSolder
- U1: footprint (none) -> Package_SO:TSSOP-28_4.4x9.7mm_P0.65mm
- U2: LCSC Part (none) -> C94590
- U5: footprint (none) -> Package_SO:SOIC-8_3.9x4.9mm_P1.27mm
- renumbered R7 to R11, R12 to R16, R1 to R2, R19 to R23, R20 to R24, R26 to R30, R28 to R32, R33 to R37, R36 to R40, R37 to R41, R38 to R42, R39 to R43, R40 to R44, R41 to R45, R42 to R46, R43 to R47, R44 to R48, R45 to R49, R46 to R50, R47 to R51, R48 to R52, R49 to R53, R50 to R54, R51 to R55, R52 to R56, R53 to R57, R4 to R7, R5 to R8, TP1 to TP2, TP2 to TP3, TP3 to TP4, TP4 to TP5, TP5 to TP6, TP6 to TP7, TP7 to TP8, TP8 to TP9
Connections:
- net GND: now also R1.2, R5.2; no longer R4.2
- net at C11.1, R40.2, R43.1: now also U5.7; no longer U5.1
- net at C11.2, R42.2: now also U5.5 (+); no longer U5.3 (+)
- net at C26.1, R44.2, R48.1: now also U5.1; no longer U5.7
- net at C26.2, R47.2: now also U5.3 (+); no longer U5.5 (+)
- net at C1.2: now also T1.1
- net at J1.3: now also T1.4
- net at R4.1: now also R1.1, R3.1, T1.8; no longer U1.20 (RXIN)
- net at U1.18 (BFRAME): now also TP1.1
- new net: R3.2, R9.2, U1.20 (RXIN)
- new net: R4.2, R5.1, R9.1, T1.5
Other:
- moved on the sheet: R4, U1B, U5A, U5B

Commit message: layout update
Parts:
- added C39, C46: 100u, Capacitor_SMD:CP_Elec_6.3x7.7, symbol Device:C_Polarized_Small
- added J4, J5: TestPoint_Small, TestPoint:TestPoint_THTPad_D2.0mm_Drill1.0mm, symbol Connector:TestPoint_Small
- R32, R37: footprint Resistor_SMD:R_0805_2012Metric_Pad1.20x1.40mm_HandSolder -> Resistor_SMD:R_0603_1608Metric_Pad0.98x0.95mm_HandSolder
- TP1, TP2, TP3, TP4, TP5, TP6, TP7, TP8, TP9: footprint TestPoint:TestPoint_Pad_D1.5mm -> TestPoint:TestPoint_Pad_D1.0mm
- U3: LCSC Part (none) -> C962089
- renumbered C39 to C40, C40 to C41, C41 to C42, C42 to C43, C43 to C44, C44 to C45, C45 to C47, J4 to J6
Connections:
- net +3.3V: now also C39.1
- net +5V: now also C46.1
- net Earth: now also J4.1, J5.1
- net GND: now also C39.2, C46.2
- net XLR_R_+: now also C12.1, J3.2; no longer C28.1, J3.3
- net XLR_R_-: now also C28.1, J3.3; no longer C12.1, J3.2
- net VIN: now reaches C32.1, J6.2, J6.3, L1.1, L2.1
- net VOUTR+: now reaches R46.1
- net VOUTR+: now also U3.13 (VOUTR+); no longer U3.14 (VOUTR-)
- net VOUTL-: now reaches R7.1, U3.11 (VOUTL-)
- net VOUTL+: now reaches R23.1, U3.12 (VOUTL+)
- net VOUTR-: now reaches R41.1
- net VOUTR-: now also U3.14 (VOUTR-); no longer U3.13 (VOUTR+)
Other:
- moved on the sheet: C23, C24

Commit message: layout update
Parts:
- removed FB2: ~, Resistor_SMD:R_0805_2012Metric_Pad1.20x1.40mm_HandSolder, symbol Device:FerriteBead_Small
- added D1: LED, LED_THT:LED_D3.0mm_Horizontal_O3.81mm_Z6.0mm, symbol Device:LED
- added Q1: BC857, Package_TO_SOT_SMD:SOT-23, symbol Transistor_BJT:BC857
- added R51, R52: 0R, Resistor_SMD:R_0805_2012Metric_Pad1.20x1.40mm_HandSolder, symbol Device:R_Small
- added R55: 1k, Resistor_SMD:R_0603_1608Metric_Pad0.98x0.95mm_HandSolder, symbol Device:R_Small
- added R57: 220R, Resistor_SMD:R_0805_2012Metric_Pad1.20x1.40mm_HandSolder, symbol Device:R_Small
- SW1: footprint (none) -> Button_Switch_SMD:SW_DIP_SPSTx01_Slide_6.7x4.1mm_W6.73mm_P2.54mm_LowProfile_JPin; LCSC Part (none) -> C19272173
- renumbered C24 to C23, C23 to C24, FB3 to FB2, FB4 to FB3, R52 to R53, R53 to R54, R51 to R56, R54 to R58, R55 to R59, R56 to R60, R57 to R61
Connections:
- net +3.3V: now also Q1.2 (E)
- net +5V: now also C17.2, C18.2, C19.2, C20.2, U3.16 (VCC2), U3.8 (VCC1)
- net Earth: now also R51.2, R52.2; no longer SW1.1
- net GND: now also SW1.1, R51.1, R52.1, R57.1
- net RSTN: now also R55.2
- net EARTH_AES: now reaches J1.1, SW1.2
- new net: Q1.1 (B), R55.1
- new net: D1.1 (K), R57.2
- new net: D1.2 (A), Q1.3 (C)
Other:
- moved on the sheet: R56, SW1

Commit message: Added Gerbers and did some improvements
Parts:
- removed Q1: BC857, Package_TO_SOT_SMD:SOT-23, symbol Transistor_BJT:BC857
- added D1, D2, D3, D4: PESD5V0U1UB, Diode_SMD:D_SOD-523, symbol SimonLib:PESD5V0U1UB
- added D6: PMEG4010CEH, Diode_SMD:D_SOD-123F, symbol Diode:PMEG4010CEH
- added Q1: BC847, Package_TO_SOT_SMD:SOT-23, symbol Transistor_BJT:BC847
- C6: footprint Capacitor_SMD:C_1206_3216Metric_Pad1.33x1.80mm_HandSolder -> Capacitor_SMD:C_0805_2012Metric_Pad1.18x1.45mm_HandSolder
- renumbered C33 to C32, C34 to C33, C32 to C34, D1 to D5, R51 to R49, R49 to R50, R50 to R51, R56 to R53, R53 to R54, R54 to R55, R57 to R56, R55 to R57
Connections:
- net +3.3V: now also D5.2 (A)
- net GND: now also D1.2, D2.2, D3.2, D4.2, Q1.2 (E); no longer R56.1
- net VIN: now also D6.1 (K); no longer J6.2, J6.3
- net at R57.1: now also Q1.1 (B)
- net at C12.2, R43.2: now also D3.1
- net at C28.2, R48.2: now also D4.1
- net at C3.2, R11.2: now also D1.1
- net at C8.2, R30.2: now also D2.1
- new net: Q1.3 (C), R56.1
- new net: D6.2 (A), J6.2, J6.3
Other:
- moved on the sheet: C31, C32, C33, C34, C35, C36, C37, C38, C39, C40, C41, C42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
